File: snrf/hw/dongle/eagle/main.sch (EAGLE design)
At the start: 12 parts, among them IC1 FT232RL, U1 ADP3338AKCZ-2.5RL7

Commit message: [ update ] schematics done, board routed. nrf connector has to be moved for fitting
Connections:
- net NRF_AM: now also PCB1.8; no longer PCB1.5
- net NRF_CD: now also PCB1.7; no longer PCB1.8
- net NRF_PWR: now also PCB1.5; no longer PCB1.7
Changed lines of the file:
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@@
 <setting verticaltext="up"/>
 </settings>
-<grid distance="2.54" unitdist="mm" unit="mm" style="lines" multiple="1" display="yes" altdistance="0.01" altunitdist="inch" altunit="inch"/>
+<grid distance="0.1" unitdist="inch" unit="inch" style="lines" multiple="1" display="yes" altdistance="0.01" altunitdist="inch" altunit="inch"/>
 <layers>
 <layer number="1" name="Top" color="4" fill="1" visible="no" active="no"/>
@@
 </segment>
 <segment>
+<pinref part="PCB1" gate="G$1" pin="8"/>
+<wire x1="5.08" y1="55.88" x2="-10.16" y2="55.88" width="0.1524" layer="91"/>
+<label x="-10.16" y="55.88" size="1.778" layer="95"/>
+</segment>
+</net>
+<net name="NRF_MISO" class="0">
+<segment>
+<pinref part="CON_NRF" gate="G$1" pin="6"/>
+<wire x1="91.44" y1="78.74" x2="76.2" y2="78.74" width="0.1524" layer="91"/>
+<label x="76.2" y="78.74" size="1.778" layer="95"/>
+</segment>
+<segment>
+<pinref part="PCB1" gate="G$1" pin="A3"/>
+<wire x1="35.56" y1="71.12" x2="53.34" y2="71.12" width="0.1524" layer="91"/>
+<label x="38.1" y="71.12" size="1.778" layer="95"/>
+</segment>
+</net>
+<net name="NRF_SCK" class="0">
+<segment>
+<pinref part="CON_NRF" gate="G$1" pin="4"/>
+<wire x1="91.44" y1="76.2" x2="76.2" y2="76.2" width="0.1524" layer="91"/>
+<label x="76.2" y="76.2" size="1.778" layer="95"/>
+</segment>
+<segment>
+<pinref part="PCB1" gate="G$1" pin="A1"/>
+<wire x1="35.56" y1="66.04" x2="53.34" y2="66.04" width="0.1524" layer="91"/>
+<label x="38.1" y="66.04" size="1.778" layer="95"/>
+</segment>
+</net>
+<net name="NRF_CSN" class="0">
+<segment>
+<pinref part="CON_NRF" gate="G$1" pin="3"/>
+<wire x1="106.68" y1="76.2" x2="121.92" y2="76.2" width="0.1524" layer="91"/>
+<label x="109.22" y="76.2" size="1.778" layer="95"/>
+</segment>
+<segment>
+<pinref part="PCB1" gate="G$1" pin="A0"/>
+<wire x1="35.56" y1="63.5" x2="53.34" y2="63.5" width="0.1524" layer="91"/>
+<label x="38.1" y="63.5" size="1.778" layer="95"/>
+</segment>
+</net>
+<net name="NRF_MOSI" class="0">
+<segment>
+<pinref part="CON_NRF" gate="G$1" pin="5"/>
+<wire x1="106.68" y1="78.74" x2="121.92" y2="78.74" width="0.1524" layer="91"/>
+<label x="109.22" y="78.74" size="1.778" layer="95"/>
+</segment>
+<segment>
+<pinref part="PCB1" gate="G$1" pin="A2"/>
+<wire x1="35.56" y1="68.58" x2="53.34" y2="68.58" width="0.1524" layer="91"/>
+<label x="38.1" y="68.58" size="1.778" layer="95"/>
+</segment>
+</net>
+<net name="NRF_DR" class="0">
+<segment>
+<pinref part="CON_NRF" gate="G$1" pin="7"/>
+<wire x1="106.68" y1="81.28" x2="121.92" y2="81.28" width="0.1524" layer="91"/>
+<label x="109.22" y="81.28" size="1.778" layer="95"/>
+</segment>
+<segment>
+<pinref part="PCB1" gate="G$1" pin="2"/>
+<wire x1="5.08" y1="71.12" x2="-10.16" y2="71.12" width="0.1524" layer="91"/>
+<label x="-10.16" y="71.12" size="1.778" layer="95"/>
+</segment>
+</net>
+<net name="NRF_CD" class="0">
+<segment>
+<pinref part="CON_NRF" gate="G$1" pin="9"/>
+<wire x1="106.68" y1="83.82" x2="121.92" y2="83.82" width="0.1524" layer="91"/>
+<label x="109.22" y="83.82" size="1.778" layer="95"/>
+</segment>
+<segment>
+<pinref part="PCB1" gate="G$1" pin="7"/>
+<wire x1="5.08" y1="58.42" x2="-10.16" y2="58.42" width="0.1524" layer="91"/>
+<label x="-10.16" y="58.42" size="1.778" layer="95"/>
+</segment>
+</net>
+<net name="NRF_PWR" class="0">
+<segment>
+<pinref part="CON_NRF" gate="G$1" pin="11"/>
+<wire x1="106.68" y1="86.36" x2="121.92" y2="86.36" width="0.1524" layer="91"/>
+<label x="109.22" y="86.36" size="1.778" layer="95"/>
+</segment>
+<segment>
 <pinref part="PCB1" gate="G$1" pin="5"/>
 <wire x1="5.08" y1="63.5" x2="-10.16" y2="63.5" width="0.1524" layer="91"/>
@@
 </segment>
 </net>
-<net name="NRF_MISO" class="0">
-<segment>
-<pinref part="CON_NRF" gate="G$1" pin="6"/>
-<wire x1="91.44" y1="78.74" x2="76.2" y2="78.74" width="0.1524" layer="91"/>
-<label x="76.2" y="78.74" size="1.778" layer="95"/>
-</segment>
-<segment>
-<pinref part="PCB1" gate="G$1" pin="A3"/>
-<wire x1="35.56" y1="71.12" x2="53.34" y2="71.12" width="0.1524" layer="91"/>
-<label x="38.1" y="71.12" size="1.778" layer="95"/>
-</segment>
-</net>
-<net name="NRF_SCK" class="0">
-<segment>
-<pinref part="CON_NRF" gate="G$1" pin="4"/>
-<wire x1="91.44" y1="76.2" x2="76.2" y2="76.2" width="0.1524" layer="91"/>
-<label x="76.2" y="76.2" size="1.778" layer="95"/>
-</segment>
-<segment>
-<pinref part="PCB1" gate="G$1" pin="A1"/>
-<wire x1="35.56" y1="66.04" x2="53.34" y2="66.04" width="0.1524" layer="91"/>
-<label x="38.1" y="66.04" size="1.778" layer="95"/>
-</segment>
-</net>
-<net name="NRF_CSN" class="0">
-<segment>
-<pinref part="CON_NRF" gate="G$1" pin="3"/>
-<wire x1="106.68" y1="76.2" x2="121.92" y2="76.2" width="0.1524" layer="91"/>
-<label x="109.22" y="76.2" size="1.778" layer="95"/>
-</segment>
-<segment>
-<pinref part="PCB1" gate="G$1" pin="A0"/>
-<wire x1="35.56" y1="63.5" x2="53.34" y2="63.5" width="0.1524" layer="91"/>
-<label x="38.1" y="63.5" size="1.778" layer="95"/>
-</segment>
-</net>
-<net name="NRF_MOSI" class="0">
-<segment>
-<pinref part="CON_NRF" gate="G$1" pin="5"/>
-<wire x1="106.68" y1="78.74" x2="121.92" y2="78.74" width="0.1524" layer="91"/>
-<label x="109.22" y="78.74" size="1.778" layer="95"/>
-</segment>
-<segment>
-<pinref part="PCB1" gate="G$1" pin="A2"/>
-<wire x1="35.56" y1="68.58" x2="53.34" y2="68.58" width="0.1524" layer="91"/>
-<label x="38.1" y="68.58" size="1.778" layer="95"/>
-</segment>
-</net>
-<net name="NRF_DR" class="0">
-<segment>
-<pinref part="CON_NRF" gate="G$1" pin="7"/>
-<wire x1="106.68" y1="81.28" x2="121.92" y2="81.28" width="0.1524" layer="91"/>
-<label x="109.22" y="81.28" size="1.778" layer="95"/>
-</segment>
-<segment>
-<pinref part="PCB1" gate="G$1" pin="2"/>
-<wire x1="5.08" y1="71.12" x2="-10.16" y2="71.12" width="0.1524" layer="91"/>
-<label x="-10.16" y="71.12" size="1.778" layer="95"/>
-</segment>
-</net>
-<net name="NRF_CD" class="0">
-<segment>
-<pinref part="CON_NRF" gate="G$1" pin="9"/>
-<wire x1="106.68" y1="83.82" x2="121.92" y2="83.82" width="0.1524" layer="91"/>
-<label x="109.22" y="83.82" size="1.778" layer="95"/>
-</segment>
-<segment>
-<pinref part="PCB1" gate="G$1" pin="8"/>
-<wire x1="5.08" y1="55.88" x2="-10.16" y2="55.88" width="0.1524" layer="91"/>
-<label x="-10.16" y="55.88" size="1.778" layer="95"/>
-</segment>
-</net>
-<net name="NRF_PWR" class="0">
-<segment>
-<pinref part="CON_NRF" gate="G$1" pin="11"/>
-<wire x1="106.68" y1="86.36" x2="121.92" y2="86.36" width="0.1524" layer="91"/>
-<label x="109.22" y="86.36" size="1.778" layer="95"/>
-</segment>
-<segment>
-<pinref part="PCB1" gate="G$1" pin="7"/>
-<wire x1="5.08" y1="58.42" x2="-10.16" y2="58.42" width="0.1524" layer="91"/>
-<label x="-10.16" y="58.42" size="1.778" layer="95"/>
-</segment>
-</net>

Commit message: [ update ] clean tNames
Parts:
- U1: value ADP3338AKCZ-2.5RL7 -> LDO33
Changed lines of the file:
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@@
 <setting verticaltext="up"/>
 </settings>
-<grid distance="0.1" unitdist="inch" unit="inch" style="lines" multiple="1" display="yes" altdistance="0.01" altunitdist="inch" altunit="inch"/>
+<grid distance="2.54" unitdist="mm" unit="mm" style="lines" multiple="1" display="yes" altdistance="0.01" altunitdist="inch" altunit="inch"/>
 <layers>
 <layer number="1" name="Top" color="4" fill="1" visible="no" active="no"/>
@@
 <part name="C3" library="resistor" deviceset="CPOL-EU" device="A/3216-18W" value="2.2u"/>
 <part name="C4" library="resistor" deviceset="CPOL-EU" device="A/3216-18W" value="2.2u"/>
-<part name="U1" library="ADP3338AKCZ" deviceset="ADP3338AKCZ-2.5RL7" device=""/>
+<part name="U1" library="ADP3338AKCZ" deviceset="ADP3338AKCZ-2.5RL7" device="" value="LDO33"/>
 <part name="C5" library="rcl" deviceset="C-EU" device="C1206K" value="100n"/>
 <part name="C6" library="resistor" deviceset="CPOL-EU" device="A/3216-18W" value="2.2u"/>
@@
 <text x="55.88" y="55.88" size="1.778" layer="97">pb3 (spi_mosi)</text>
 <text x="55.88" y="53.34" size="1.778" layer="97">pb2 (spi_csn)</text>
-<text x="-38.1" y="5.08" size="1.778" layer="97">actually a ap1117e33g</text>
+<text x="-45.72" y="7.62" size="1.778" layer="97">actually a ap1117e33g</text>
 </plain>
 <instances>
 <instance part="PCB1" gate="G$1" x="20.32" y="63.5" rot="R90"/>
-<instance part="CON_NRF" gate="G$1" x="99.06" y="81.28"/>
+<instance part="CON_NRF" gate="G$1" x="99.06" y="81.28" smashed="yes">
+<attribute name="VALUE" x="95.25" y="68.58" size="1.778" layer="96"/>
+<attribute name="NAME" x="92.71" y="66.802" size="1.778" layer="95"/>
+</instance>
 <instance part="CON_HOST_SPI" gate="1" x="-55.88" y="81.28"/>
 <instance part="CON_HOST_USB" gate="G$1" x="-55.88" y="50.8" rot="R180"/>
@@
 <instance part="C3" gate="G$1" x="-63.5" y="15.24"/>
 <instance part="C4" gate="G$1" x="2.54" y="12.7"/>
-<instance part="U1" gate="A" x="-33.02" y="20.32"/>
+<instance part="U1" gate="A" x="-33.02" y="20.32" smashed="yes">
+<attribute name="NAME" x="-37.7444" y="27.0764" size="2.0828" layer="95" ratio="10" rot="SR0"/>
+<attribute name="VALUE" x="-38.735" y="7.5438" size="2.0828" layer="96" ratio="10" rot="SR0" display="off"/>
+</instance>
 <instance part="C5" gate="G$1" x="58.42" y="35.56"/>
 <instance part="C6" gate="G$1" x="50.8" y="35.56"/>
